File: Water-Probe/Design Files/EDA/BoSL Probe/BoSL Probe.sch (KiCad schematic (older format))
At the start: 9 parts, among them J1 8P8C_Shielded, U1 MS5803-01BA, U2 DS18B20

Commit message: commiting pcb changes for probe
Parts:
- C1: footprint Capacitors_SMD:C_0603_HandSoldering -> Capacitors_SMD:C_0805_HandSoldering
- H1, H2: footprint Mounting_Holes:MountingHole_3.2mm_M3 -> Measurement_Points:Measurement_Point_Round-TH_Big
- R1, R2, R3: footprint Resistors_SMD:R_0603_HandSoldering -> Resistors_SMD:R_0805_HandSoldering
- U2: footprint TO_SOT_Packages_THT:TO-92_Inline_Narrow_Oval -> TO_SOT_Packages_THT:TO-92_Horizontal2_Inline_Narrow_Oval
Changed lines of the file:
@@
 F 0 "C1" H 3065 4945 50  0000 L CNN
 F 1 "100nF" H 3065 4856 50  0000 L CNN
-F 2 "Capacitors_SMD:C_0603_HandSoldering" H 2988 4750 50  0001 C CNN
+F 2 "Capacitors_SMD:C_0805_HandSoldering" H 2988 4750 50  0001 C CNN
 F 3 "~" H 2950 4900 50  0001 C CNN
 	1    2950 4900
@@
 F 0 "R1" H 4550 4750 50  0000 L CNN
 F 1 "10 kΩ" H 4400 4650 50  0000 L CNN
-F 2 "Resistors_SMD:R_0603_HandSoldering" V 4630 4700 50  0001 C CNN
+F 2 "Resistors_SMD:R_0805_HandSoldering" V 4630 4700 50  0001 C CNN
 F 3 "~" H 4700 4700 50  0001 C CNN
 	1    4700 4700
@@
 F 0 "R2" H 4550 5150 50  0000 L CNN
 F 1 "10 kΩ" H 4400 5050 50  0000 L CNN
-F 2 "Resistors_SMD:R_0603_HandSoldering" V 4630 5100 50  0001 C CNN
+F 2 "Resistors_SMD:R_0805_HandSoldering" V 4630 5100 50  0001 C CNN
 F 3 "~" H 4700 5100 50  0001 C CNN
 	1    4700 5100
@@
 F 0 "U2" H 5320 3345 50  0000 R CNN
 F 1 "DS18B20" H 5320 3256 50  0000 R CNN
-F 2 "TO_SOT_Packages_THT:TO-92_Inline_Narrow_Oval" H 4550 3050 50  0001 C CNN
+F 2 "TO_SOT_Packages_THT:TO-92_Horizontal2_Inline_Narrow_Oval" H 4550 3050 50  0001 C CNN
 F 3 "http://datasheets.maximintegrated.com/en/ds/DS18B20.pdf" H 5400 3550 50  0001 C CNN
 	1    5550 3300
@@
 F 0 "R3" H 6070 3195 50  0000 L CNN
 F 1 "4.7 kΩ" H 6070 3106 50  0000 L CNN
-F 2 "Resistors_SMD:R_0603_HandSoldering" V 5930 3150 50  0001 C CNN
+F 2 "Resistors_SMD:R_0805_HandSoldering" V 5930 3150 50  0001 C CNN
 F 3 "~" H 6000 3150 50  0001 C CNN
 	1    6000 3150
@@
 F 0 "H1" H 7450 3750 50  0000 L CNN
 F 1 "MountingHole_Pad" H 6900 3650 50  0000 L CNN
-F 2 "Mounting_Holes:MountingHole_3.2mm_M3" H 7500 3450 50  0001 C CNN
+F 2 "Measurement_Points:Measurement_Point_Round-TH_Big" H 7500 3450 50  0001 C CNN
 F 3 "~" H 7500 3450 50  0001 C CNN
 	1    7500 3450
@@
 F 0 "H2" H 8000 3750 50  0000 L CNN
 F 1 "MountingHole_Pad" H 8000 3650 50  0000 L CNN
-F 2 "Mounting_Holes:MountingHole_3.2mm_M3" H 8050 3450 50  0001 C CNN
+F 2 "Measurement_Points:Measurement_Point_Round-TH_Big" H 8050 3450 50  0001 C CNN
 F 3 "~" H 8050 3450 50  0001 C CNN
 	1    8050 3450
