File: Water-Probe/Design Files/EDA/BoSL Probe/_autosave-BoSL Probe.sch (KiCad schematic (older format))
At the start: 9 parts, among them J1 8P8C_Shielded, U1 MS5803-01BA, U2 DS18B20

Commit message: keystone rightangle screw connectors added
Parts:
- gave numbers to parts that had none: 2
Changed lines of the file:
@@
 $EndComp
 $Comp
-L Project:KeyStone_Screw J?
+L Project:KeyStone_Screw J3
 U 1 1 5D953E64
 P 8050 3100
-F 0 "J?" V 8238 3187 50  0000 L CNN
+F 0 "J3" V 8238 3187 50  0000 L CNN
 F 1 "KeyStone_Screw" V 8327 3187 50  0000 L CNN
 F 2 "Project:KeyStone_Screw" H 8050 3100 50  0001 C CNN
@@
 $EndComp
 $Comp
-L Project:KeyStone_Screw J?
+L Project:KeyStone_Screw J2
 U 1 1 5D9540DF
 P 7500 3100
-F 0 "J?" V 7688 3187 50  0000 L CNN
+F 0 "J2" V 7688 3187 50  0000 L CNN
 F 1 "KeyStone_Screw" V 7777 3187 50  0000 L CNN
 F 2 "Project:KeyStone_Screw" H 7500 3100 50  0001 C CNN
