File: Board-Hardware/EDA BoSLGPS/BoSL_GSP.kicad_pcb (KiCad board)
At the start: 2 copper layers, 88 x 69.8 mm, 58 parts, among them CON1 Micro_SD_Card, CON2 BARREL_JACK, IC1 ATMEGA328-P, IC2 SIM7000, J1 Screw_Terminal_1x06, J2 Screw_Terminal_1x04, J3 Screw_Terminal_1x02, J4 Screw_Terminal_1x08, J5 Screw_Terminal_1x04, J6 RJ45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

Commit message: generated bosl gsp gerber files and bom
Routing:
- net GND: vias 27 -> 28
Changed lines of the file:
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@@
     (thickness 1.6)
     (drawings 117)
-    (tracks 967)
+    (tracks 968)
     (zones 0)
     (modules 58)
@@
       (drillshape 0)
       (scaleselection 1)
-      (outputdirectory "../Production Files/Gerber/"))
+      (outputdirectory "../Manufacturing/Gerber GSP/"))
   )
   (net 0 "")
@@
   (gr_arc (start 190.5 130.8) (end 190.5 132.8) (angle -90) (layer Edge.Cuts) (width 0.15))
   (gr_arc (start 190.5 65) (end 192.5 65) (angle -90) (layer Edge.Cuts) (width 0.15))
-  (segment (start 183.7 70.92) (end 183.7 69.75) (width 3.23) (layer F.Cu) (net 57))
   (via (at 185.9 68.8) (size 0.6) (drill 0.4) (layers F.Cu B.Cu) (net 1))
   (via (at 181.5 68.7) (size 0.6) (drill 0.4) (layers F.Cu B.Cu) (net 1))
@@
   (segment (start 128.8 103.275) (end 128.8 106.125) (width 0.4) (layer F.Cu) (net 1))
   (via (at 111.6 106.2) (size 0.6) (drill 0.4) (layers F.Cu B.Cu) (net 1))
+  (via (at 182.8 82) (size 0.6) (drill 0.4) (layers F.Cu B.Cu) (net 1))
   (segment (start 176.69 77.92) (end 176.69 75.31) (width 0.6) (layer F.Cu) (net 2) (status 10))
   (segment (start 176.69 75.31) (end 176.69 73.914202) (width 3.23) (layer F.Cu) (net 2))
@@
   (segment (start 156.733 83.133) (end 153.786 83.133) (width 0.25) (layer F.Cu) (net 56) (status 20))
   (segment (start 158.8 85.2) (end 156.733 83.133) (width 0.25) (layer F.Cu) (net 56))
+  (segment (start 183.7 70.92) (end 183.7 69.75) (width 3.23) (layer F.Cu) (net 57))
   (segment (start 183.7 77.91) (end 183.69 77.92) (width 0.6) (layer F.Cu) (net 58))
   (segment (start 183.7 75.18) (end 183.7 75.25) (width 3.23) (layer F.Cu) (net 58))
