File: Velocity/EDA/AM Demodulator/AM Demodulator/AM Demodulator.sch (KiCad schematic (older format))
At the start: 22 parts

Commit message: added velocity AM demodulator gerbers
Parts:
- removed J? (x2): Receiver In, symbol Connector_Generic:Conn_01x01
- removed J? (x2): Emmiter In, symbol Connector_Generic:Conn_01x01
- added J2: Conn_01x02, Pin_Headers:Pin_Header_Straight_1x02_Pitch2.54mm, symbol Connector_Generic:Conn_01x02
- C1, C2: renamed from C?; footprint (none) -> Capacitors_THT:CP_Radial_D5.0mm_P2.50mm
- D1: renamed from D?; footprint Diode_THT:D_DO-35_SOD27_P7.62mm_Horizontal -> Diodes_THT:D_A-405_P7.62mm_Horizontal
- J1, J6: renamed from J?; footprint (none) -> Pin_Headers:Pin_Header_Straight_1x01_Pitch2.54mm
- LS1, LS2: renamed from LS?; footprint (none) -> Pin_Headers:Pin_Header_Straight_1x02_Pitch2.54mm
- R1, R2, R3, R4, R5, R6, R7, R8: renamed from R?; footprint (none) -> Resistors_THT:R_Axial_DIN0204_L3.6mm_D1.6mm_P7.62mm_Horizontal
- U1: renamed from U?; footprint (none) -> Housings_DIP:DIP-8_W7.62mm_LongPads
Connections:
- net GND: now also J2.1 (Pin_1)
- net VPP: now also J2.2 (Pin_2)

Commit message: daily commit
Parts:
- C1: value 1 μF -> 100 nF
Changed lines of the file:
@@
 P 4600 4150
 F 0 "C1" H 4715 4195 50  0000 L CNN
-F 1 "1 μF" H 4715 4106 50  0000 L CNN
+F 1 "100 nF" H 4715 4106 50  0000 L CNN
 F 2 "Capacitors_THT:CP_Radial_D5.0mm_P2.50mm" H 4638 4000 50  0001 C CNN
 F 3 "~" H 4600 4150 50  0001 C CNN
