File: Velocity/Heterodyne/EDA/Heterodyne/Heterodyne.sch (KiCad schematic (older format))
At the start: 36 parts, among them J1 OP_IN, J2 OP_OUT, J3 PWR, J4 Doppler_Out, J5 V_Square, U1 SA612AD, U2 NE5532

Commit message: added bom and pcb files for velocity sensor
Parts:
- removed C?: 100 nF, Capacitors_SMD:C_0805_HandSoldering, symbol Device:C
- removed R10: 1 kΩ, Resistors_SMD:R_0805_HandSoldering, symbol Device:R
- added C14: 1 μF, Capacitors_SMD:C_1206_HandSoldering, symbol Device:C
- added C4, C5, C6: 100 nF, Capacitors_SMD:C_0805_HandSoldering, symbol Device:C
- added J6: OP_OUT, Pin_Headers:Pin_Header_Straight_1x02_Pitch2.54mm, symbol Connector_Generic:Conn_01x02
- added R3: 10 kΩ, Resistors_SMD:R_0805_HandSoldering, symbol Device:R
- C10, C12, C9: renamed from C?; footprint (none) -> Capacitors_SMD:C_0805_HandSoldering
- C11: renamed from C?; footprint (none) -> Capacitors_SMD:CP_Elec_8x10
- C13: renamed from C?; footprint (none) -> Capacitors_SMD:C_1206_HandSoldering
- C3, C7: value 680 pF -> 100 nF
- J7, J8: renamed from J?; footprint (none) -> Pin_Headers:Pin_Header_Straight_1x01_Pitch2.54mm
- R1, R4: value 3.3 kΩ -> 10 kΩ
- R5: value 2.2 kΩ -> 10 kΩ
- R6: value 1 kΩ -> 10 kΩ
- R7, R8: value 330 kΩ -> 10 kΩ
- R9: value 2.2 kΩ -> 39 kΩ
- U3: renamed from U?; footprint Package_TO_SOT_SMD:SOT-323_SC-70 -> TO_SOT_Packages_SMD:SOT-323_SC-70_Handsoldering
- gave numbers to parts that had none: 1
Connections:
- net GND: now also C14.2, J6.1 (Pin_1); no longer R4.2, R8.2
- net VPP: now also C14.1; no longer R1.1, R7.1
- net at U1.4 (OUT_A): now also JP1.2
- net at U1.5 (OUT_B): now also R6.1; no longer JP1.2
- net at R7.2, U2.5 (+): now also C7.1; no longer R8.1
- net at JP2.3, U2.7: now also R9.2, C6.2; no longer C7.1, R9.1
- net at JP1.1: now also C7.2, R8.1
- net at C3.2, R5.2: now also R1.2, U2.1, C5.2, J6.2 (Pin_2); no longer R6.2, U2.2 (-)
- net at J1.1 (Pin_1): now also R4.1; no longer R6.1
- new net: R8.2, R9.1, U2.6 (-)
- new net: C4.2, C5.1, R4.2, R5.1, U2.2 (-)
- new net: C3.1, C4.1, R1.1, R3.2, U2.3 (+)
- new net: J2.2 (Pin_2), R3.1
- new net: C6.1, R6.2, R7.1
Other:
- moved on the sheet: C1, C10, C11, C12, C13, C2, C8, C9, J1, J2, J3, J4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
