File: Velocity/Heterodyne/EDA/Heterodyne/Heterodyne.kicad_pcb (KiCad board)
At the start: 4 copper layers, 35.5 x 19 mm, 37 parts, among them J1 Conn_01x05, J7 Reciever, U1 SA612AD, U2 NE5532DR, U3 MAX7375AXR105, U4 MAX11613, U5 ATmega328PB-AU, Y1 8 MHz

Commit message: finished bosl board rev0.4 layout
Parts:
- added C7: 100 nF, Capacitor_SMD:C_0603_1608Metric_Pad1.05x0.95mm_HandSolder, F.Cu at (108.8, 59.9)
- J1: value Conn_01x05 -> Conn_01x06; footprint Connector_PinHeader_2.54mm:PinHeader_1x05_P2.54mm_Vertical -> Connector_PinHeader_2.54mm:PinHeader_1x06_P2.54mm_Vertical
Connections:
- R5 pad 1: VPP -> VREF
- U5 pad 23: Net-(U5-Pad23) -> VREF
- U5 pad 32: Net-(U5-Pad32) -> TLL_WAKE
Routing:
- net VREF: track 0.00 -> 18.6 mm, vias 0 -> 1
- net TLL_WAKE: track 0.00 -> 9.50 mm
- net GND: track 38.2 -> 41.1 mm
- net VPP: track 27.9 -> 25.6 mm, vias 5 -> 4
- net Net-(C7-Pad1): track 3.46 -> 5.11 mm
Other:
- board text added: "BoSL Velocity rev 0.1.1"
- board text added: "WKE"
- board text removed: "BoSL Velocity rev 0.1"
