File: Board-Hardware/EDA/BoSL.sch (KiCad schematic (older format))
At the start: 62 parts, among them CON1 Micro_SD_Card, CON2 BARREL_JACK, IC2 SIM7000, J1 Screw_Terminal_1x06, J2 Screw_Terminal_1x04, J3 Screw_Terminal_1x02, J4 Screw_Terminal_1x08, J5 Screw_Terminal_1x04, J6 RJ45, J7 USB_B_Micro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

Commit message: added  update layout for bosl v4
Parts:
- AT1: footprint Connectors:SMA_THT_Jack_Straight -> Connector_Coaxial:SMA_Amphenol_901-144_Vertical
- AT2: footprint Connectors_Molex:Molex_Microcoaxial_RF -> Connector_Coaxial:U.FL_Molex_MCRF_73412-0110_Vertical
- C7: footprint Capacitors_SMD:CP_Elec_8x10 -> Capacitor_SMD:CP_Elec_8x10
- CON2: footprint Connectors:BARREL_JACK -> Connector_BarrelJack:BarrelJack_Horizontal
- D1: footprint Diodes_SMD:D_SOD-323_HandSoldering -> Diode_SMD:D_SOD-323
- H1, H2: footprint Mounting_Holes:MountingHole_2.2mm_M2 -> MountingHole:MountingHole_2.2mm_M2_Pad
- J1: footprint SIMFootprints:Screw_Terminals_1x6 -> TerminalBlock_Phoenix:TerminalBlock_Phoenix_MKDS-1,5-6_1x06_P5.00mm_Horizontal
- J2, J5: footprint SIMFootprints:Screw_Terminals_1x4 -> TerminalBlock_Phoenix:TerminalBlock_Phoenix_MKDS-1,5-4_1x04_P5.00mm_Horizontal
- J3: footprint SIMFootprints:Screw_Terminals_1x2 -> TerminalBlock_Phoenix:TerminalBlock_Phoenix_MKDS-1,5-2_1x02_P5.00mm_Horizontal
- J4: footprint SIMFootprints:Screw_Terminals_1x8 -> TerminalBlock_Phoenix:TerminalBlock_Phoenix_MKDS-1,5-8_1x08_P5.00mm_Horizontal
- J7: footprint Connectors:USB_Micro-B -> Connector_USB:USB_Micro-B_Molex-105017-0001
- P1: footprint Pin_Headers:Pin_Header_Straight_1x16_Pitch2.54mm -> Connector_PinHeader_2.54mm:PinHeader_1x16_P2.54mm_Vertical
- P2, P3, P4, P7: footprint Pin_Headers:Pin_Header_Straight_1x04_Pitch2.54mm -> Connector_PinHeader_2.54mm:PinHeader_1x04_P2.54mm_Vertical
- P6: footprint Pin_Headers:Pin_Header_Straight_1x09_Pitch2.54mm -> Connector_PinHeader_2.54mm:PinHeader_1x09_P2.54mm_Vertical
- P9: footprint Pin_Headers:Pin_Header_Straight_1x12_Pitch2.54mm -> Connector_PinHeader_2.54mm:PinHeader_1x12_P2.54mm_Vertical
- SW1: footprint Buttons_Switches_SMD:SW_SPST_B3S-1000 -> Button_Switch_SMD:SW_SPST_B3S-1000
- TP1, TP2, TP3: footprint Measurement_Points:Measurement_Point_Round-SMD-Pad_Small -> TestPoint:TestPoint_Pad_D1.0mm
- U1: footprint TO_SOT_Packages_SMD:SOT-89-3_Handsoldering -> Package_TO_SOT_SMD:SOT-89-3
- U3: footprint TO_SOT_Packages_SMD:SOT-353_SC-70-5_Handsoldering -> Package_TO_SOT_SMD:SOT-353_SC-70-5
- U4: footprint Housings_SOIC:SOIC-14_3.9x8.7mm_Pitch1.27mm -> Package_SO:SOIC-14_3.9x8.7mm_P1.27mm
- U5: footprint Housings_SSOP:SSOP-28_5.3x10.2mm_Pitch0.65mm -> Package_SO:SSOP-28_5.3x10.2mm_P0.65mm
- Y1: footprint Crystals:Crystal_HC49-U_Vertical -> Crystal:Crystal_HC49-4H_Vertical
Changed lines of the file:
@@
 F 0 "D1" H 5900 2150 50  0000 C CNN
 F 1 "1N4148" H 5900 1950 50  0000 C CNN
-F 2 "Diodes_SMD:D_SOD-323_HandSoldering" H 5900 2050 50  0001 C CNN
+F 2 "Diode_SMD:D_SOD-323" H 5900 2050 50  0001 C CNN
 F 3 "" H 5900 2050 50  0000 C CNN
 	1    5900 2050
@@
 F 0 "Y1" H 4550 4450 50  0000 C CNN
 F 1 "8 MHz" H 4550 4150 50  0000 C CNN
-F 2 "Crystals:Crystal_HC49-U_Vertical" H 4550 4300 50  0001 C CNN
+F 2 "Crystal:Crystal_HC49-4H_Vertical" H 4550 4300 50  0001 C CNN
 F 3 "" H 4550 4300 50  0000 C CNN
 	1    4550 4300
@@
 F 0 "CON2" H 4700 1450 50  0000 C CNN
 F 1 "BARREL_JACK" H 4700 1000 50  0000 C CNN
-F 2 "Connectors:BARREL_JACK" H 4700 1200 50  0001 C CNN
+F 2 "Connector_BarrelJack:BarrelJack_Horizontal" H 4700 1200 50  0001 C CNN
 F 3 "" H 4700 1200 50  0000 C CNN
 	1    4700 1200
@@
 F 0 "TP2" H 6550 2850 50  0000 C BNN
 F 1 "TEST" H 6550 2800 50  0000 C CNN
-F 2 "Measurement_Points:Measurement_Point_Round-SMD-Pad_Small" H 6550 2550 50  0001 C CNN
+F 2 "TestPoint:TestPoint_Pad_D1.0mm" H 6550 2550 50  0001 C CNN
 F 3 "" H 6550 2550 50  0000 C CNN
 	1    6550 2550
@@
 F 0 "P7" H 6750 5550 50  0000 C CNN
 F 1 "CONN_01X04" V 6850 5300 50  0000 C CNN
-F 2 "Pin_Headers:Pin_Header_Straight_1x04_Pitch2.54mm" H 6750 5300 50  0001 C CNN
+F 2 "Connector_PinHeader_2.54mm:PinHeader_1x04_P2.54mm_Vertical" H 6750 5300 50  0001 C CNN
 F 3 "" H 6750 5300 50  0000 C CNN
 	1    6750 5300
@@
 F 0 "TP3" H 7550 4500 50  0000 C BNN
 F 1 "TEST" H 7550 4450 50  0000 C CNN
-F 2 "Measurement_Points:Measurement_Point_Round-SMD-Pad_Small" H 7550 4200 50  0001 C CNN
+F 2 "TestPoint:TestPoint_Pad_D1.0mm" H 7550 4200 50  0001 C CNN
 F 3 "" H 7550 4200 50  0000 C CNN
 	1    7550 4200
@@
 F 0 "P3" H 1900 8900 50  0000 C CNN
 F 1 "CONN_01X04" V 2000 8650 50  0000 C CNN
-F 2 "Pin_Headers:Pin_Header_Straight_1x04_Pitch2.54mm" H 1900 8650 50  0001 C CNN
+F 2 "Connector_PinHeader_2.54mm:PinHeader_1x04_P2.54mm_Vertical" H 1900 8650 50  0001 C CNN
 F 3 "" H 1900 8650 50  0000 C CNN
 	1    1900 8650
@@
 F 0 "SW1" H 900 4600 60  0000 C CNN
 F 1 "SPST" H 900 4800 60  0000 C CNN
-F 2 "Buttons_Switches_SMD:SW_SPST_B3S-1000" H 850 4800 60  0001 C CNN
+F 2 "Button_Switch_SMD:SW_SPST_B3S-1000" H 850 4800 60  0001 C CNN
 F 3 "" H 850 4800 60  0001 C CNN
 	1    900  4700
@@
 F 0 "AT1" H 8000 750 50  0000 L CNN
 F 1 "AT" H 8000 650 50  0000 L CNN
-F 2 "Connectors:SMA_THT_Jack_Straight" H 7888 500 50  0001 C CNN
+F 2 "Connector_Coaxial:SMA_Amphenol_901-144_Vertical" H 7888 500 50  0001 C CNN
 F 3 "" H 7850 650 50  0000 C CNN
 	1    7850 650
@@
 F 0 "P4" H 1950 7350 50  0000 C CNN
 F 1 "CONN_01X04" V 2050 7100 50  0000 C CNN
-F 2 "Pin_Headers:Pin_Header_Straight_1x04_Pitch2.54mm" H 1950 7100 50  0001 C CNN
+F 2 "Connector_PinHeader_2.54mm:PinHeader_1x04_P2.54mm_Vertical" H 1950 7100 50  0001 C CNN
 F 3 "" H 1950 7100 50  0000 C CNN
 	1    1950 7100
@@
 F 0 "U3" H 8900 5450 60  0000 C CNN
 F 1 "MSQA6V1W5T2G" H 8550 5550 60  0000 C CNN
-F 2 "TO_SOT_Packages_SMD:SOT-353_SC-70-5_Handsoldering" H 8600 5750 60  0001 C CNN
+F 2 "Package_TO_SOT_SMD:SOT-353_SC-70-5" H 8600 5750 60  0001 C CNN
 F 3 "" H 8600 5750 60  0001 C CNN
 	1    8550 5750
@@
 F 0 "J1" H 1100 10450 50  0000 C TNN
 F 1 "Screw_Terminal_1x06" V 950 9800 50  0000 C TNN
-F 2 "SIMFootprints:Screw_Terminals_1x6" H 1100 9175 50  0001 C CNN
+F 2 "TerminalBlock_Phoenix:TerminalBlock_Phoenix_MKDS-1,5-6_1x06_P5.00mm_Horizontal" H 1100 9175 50  0001 C CNN
 F 3 "" H 1075 10200 50  0001 C CNN
 	1    1100 9800
@@
 F 0 "J2" H 1900 9750 50  0000 C TNN
 F 1 "Screw_Terminal_1x04" V 1750 9300 50  0000 C TNN
-F 2 "SIMFootprints:Screw_Terminals_1x4" H 1900 8875 50  0001 C CNN
+F 2 "TerminalBlock_Phoenix:TerminalBlock_Phoenix_MKDS-1,5-4_1x04_P5.00mm_Horizontal" H 1900 8875 50  0001 C CNN
 F 3 "" H 1875 9500 50  0001 C CNN
 	1    1900 9300
@@
 F 0 "P6" H 3700 7800 50  0000 C CNN
 F 1 "CONN_01X09" V 3800 7300 50  0000 C CNN
-F 2 "Pin_Headers:Pin_Header_Straight_1x09_Pitch2.54mm" H 3700 7300 50  0001 C CNN
+F 2 "Connector_PinHeader_2.54mm:PinHeader_1x09_P2.54mm_Vertical" H 3700 7300 50  0001 C CNN
 F 3 "" H 3700 7300 50  0000 C CNN
 	1    3700 7300
@@
 F 0 "TP1" H 6200 2100 50  0000 C BNN
 F 1 "TEST" H 6200 2050 50  0000 C CNN
-F 2 "Measurement_Points:Measurement_Point_Round-SMD-Pad_Small" H 6200 1800 50  0001 C CNN
+F 2 "TestPoint:TestPoint_Pad_D1.0mm" H 6200 1800 50  0001 C CNN
 F 3 "" H 6200 1800 50  0000 C CNN
 	1    6200 1800
@@
 F 0 "C7" H 9225 1450 50  0000 L CNN
 F 1 "330 μF" H 9225 1250 50  0000 L CNN
-F 2 "Capacitors_SMD:CP_Elec_8x10" H 9238 1200 50  0001 C CNN
+F 2 "Capacitor_SMD:CP_Elec_8x10" H 9238 1200 50  0001 C CNN
 F 3 "" H 9200 1350 50  0000 C CNN
 	1    9200 1350
@@
 F 0 "J4" H 3000 10350 50  0000 C TNN
 F 1 "Screw_Terminal_1x08" V 2850 9500 50  0000 C TNN
-F 2 "SIMFootprints:Screw_Terminals_1x8" H 3000 8675 50  0001 C CNN
+F 2 "TerminalBlock_Phoenix:TerminalBlock_Phoenix_MKDS-1,5-8_1x08_P5.00mm_Horizontal" H 3000 8675 50  0001 C CNN
 F 3 "" H 2975 10100 50  0001 C CNN
 	1    3000 9500
@@
 F 0 "J3" H 1950 7800 50  0000 C TNN
 F 1 "Screw_Terminal_1x02" V 1800 7550 50  0000 C TNN
-F 2 "SIMFootprints:Screw_Terminals_1x2" H 1950 7325 50  0001 C CNN
+F 2 "TerminalBlock_Phoenix:TerminalBlock_Phoenix_MKDS-1,5-2_1x02_P5.00mm_Horizontal" H 1950 7325 50  0001 C CNN
 F 3 "" H 1925 7550 50  0001 C CNN
 	1    1950 7550
@@
 F 0 "P2" H 1900 8400 50  0000 C CNN
 F 1 "CONN_01X04" V 2000 8150 50  0000 C CNN
-F 2 "Pin_Headers:Pin_Header_Straight_1x04_Pitch2.54mm" H 1900 8150 50  0001 C CNN
+F 2 "Connector_PinHeader_2.54mm:PinHeader_1x04_P2.54mm_Vertical" H 1900 8150 50  0001 C CNN
 F 3 "" H 1900 8150 50  0000 C CNN
 	1    1900 8150
@@
 F 0 "J5" H 3850 8650 50  0000 C TNN
 F 1 "Screw_Terminal_1x04" V 3700 8200 50  0000 C TNN
-F 2 "SIMFootprints:Screw_Terminals_1x4" H 3850 7775 50  0001 C CNN
+F 2 "TerminalBlock_Phoenix:TerminalBlock_Phoenix_MKDS-1,5-4_1x04_P5.00mm_Horizontal" H 3850 7775 50  0001 C CNN
 F 3 "" H 3825 8400 50  0001 C CNN
 	1    3850 8200
@@
 F 0 "P9" H 1100 8900 50  0000 C CNN
 F 1 "CONN_01X12" V 1200 8250 50  0000 C CNN
-F 2 "Pin_Headers:Pin_Header_Straight_1x12_Pitch2.54mm" H 1100 8250 50  0001 C CNN
+F 2 "Connector_PinHeader_2.54mm:PinHeader_1x12_P2.54mm_Vertical" H 1100 8250 50  0001 C CNN
 F 3 "" H 1100 8250 50  0000 C CNN
 	1    1100 8250
@@
 F 0 "P1" H 2900 8650 50  0000 C CNN
 F 1 "CONN_01X16" V 3000 7800 50  0000 C CNN
-F 2 "Pin_Headers:Pin_Header_Straight_1x16_Pitch2.54mm" H 2900 7800 50  0001 C CNN
+F 2 "Connector_PinHeader_2.54mm:PinHeader_1x16_P2.54mm_Vertical" H 2900 7800 50  0001 C CNN
 F 3 "" H 2900 7800 50  0000 C CNN
 	1    2900 7800
@@
 F 0 "J7" V 15211 3529 50  0000 L CNN
 F 1 "USB_B_Micro" V 14950 2900 50  0000 L CNN
-F 2 "Connectors:USB_Micro-B" H 15350 3150 50  0001 C CNN
+F 2 "Connector_USB:USB_Micro-B_Molex-105017-0001" H 15350 3150 50  0001 C CNN
 F 3 "~" H 15350 3150 50  0001 C CNN
 	1    15200 3200
@@
 F 0 "U5" H 14250 1300 60  0000 C CNN
 F 1 "FT232RL" H 14250 1400 60  0000 C CNN
-F 2 "Housings_SSOP:SSOP-28_5.3x10.2mm_Pitch0.65mm" H 14700 1500 60  0001 C CNN
+F 2 "Package_SO:SSOP-28_5.3x10.2mm_P0.65mm" H 14700 1500 60  0001 C CNN
 F 3 "" H 14700 1500 60  0001 C CNN
 	1    14250 1350
@@
 F 0 "U1" H 2250 900 50  0000 C CNN
 F 1 "MCP1700T-3302E/TT" H 2150 1400 50  0000 C CNN
-F 2 "TO_SOT_Packages_SMD:SOT-89-3_Handsoldering" H 2150 1200 50  0001 C CNN
+F 2 "Package_TO_SOT_SMD:SOT-89-3" H 2150 1200 50  0001 C CNN
 F 3 "" H 2150 1200 50  0000 C CNN
 	1    2150 1100
@@
 F 0 "H1" H 10100 3996 50  0000 L CNN
 F 1 "MountingHole" H 10100 3905 50  0000 L CNN
-F 2 "Mounting_Holes:MountingHole_2.2mm_M2" H 10000 3950 50  0001 C CNN
+F 2 "MountingHole:MountingHole_2.2mm_M2_Pad" H 10000 3950 50  0001 C CNN
 F 3 "~" H 10000 3950 50  0001 C CNN
 	1    10000 3950
@@
 F 0 "H2" H 10800 3996 50  0000 L CNN
 F 1 "MountingHole" H 10800 3905 50  0000 L CNN
-F 2 "Mounting_Holes:MountingHole_2.2mm_M2" H 10700 3950 50  0001 C CNN
+F 2 "MountingHole:MountingHole_2.2mm_M2_Pad" H 10700 3950 50  0001 C CNN
 F 3 "~" H 10700 3950 50  0001 C CNN
 	1    10700 3950
@@
 F 0 "U4" H 12050 1843 60  0000 C CNN
 F 1 "74HC126" H 12050 1739 60  0000 C CNN
-F 2 "Housings_SOIC:SOIC-14_3.9x8.7mm_Pitch1.27mm" H 12050 1300 60  0001 C CNN
+F 2 "Package_SO:SOIC-14_3.9x8.7mm_P1.27mm" H 12050 1300 60  0001 C CNN
 F 3 "http://www.farnell.com/datasheets/2030230.pdf?_ga=2.69642903.606851804.1567147512-325851870.1553337182&_gac=1.41560982.1567151116.EAIaIQobChMI1uyK5Yyq5AIVSSUrCh05hgU3EAkYASABEgJC2_D_BwE" H 12050 1300 60  0001 C CNN
 	1    12050 1300
@@
 F 0 "AT2" H 8700 550 50  0000 L CNN
 F 1 "AT-GNSS" H 8500 750 50  0000 L CNN
-F 2 "Connectors_Molex:Molex_Microcoaxial_RF" H 8888 500 50  0001 C CNN
+F 2 "Connector_Coaxial:U.FL_Molex_MCRF_73412-0110_Vertical" H 8888 500 50  0001 C CNN
 F 3 "" H 8850 650 50  0000 C CNN
 	1    8850 650

Commit message: added revision of bosl board
Parts:
- added BT1: Battery_Cell, SIMFootprints:2996TR, symbol Device:Battery_Cell
Connections:
- net GND: now also BT1.2 (-)
- net V_3.3: no longer U7.3 (VBAT)
- new net: BT1.1 (+), U7.3 (VBAT)
Changed lines of the file:
@@
 Text GLabel 11400 4800 1    60   Input ~ 0
-V_3.3
-Text GLabel 11500 4800 1    60   Input ~ 0
 V_3.3
 $Comp
@@
 Wire Notes Line
 	13250 6000 13250 4300
+$Comp
+L Device:Battery_Cell BT1
+U 1 1 5EA93550
+P 12150 4450
+F 0 "BT1" V 12405 4500 50  0000 C CNN
+F 1 "Battery_Cell" V 12314 4500 50  0000 C CNN
+F 2 "SIMFootprints:2996TR" V 12150 4510 50  0001 C CNN
+F 3 "LR44 KEYSTONE2996TR" V 12150 4510 50  0001 C CNN
+	1    12150 4450
+	0    -1   -1   0
+$EndComp
+Wire Wire Line
+	11950 4450 11500 4450
+Wire Wire Line
+	11500 4450 11500 4800
+$Comp
+L power:GND #PWR0102
+U 1 1 5EA9A82A
+P 12250 4450
+F 0 "#PWR0102" H 12250 4200 50  0001 C CNN
+F 1 "GND" H 12250 4300 50  0000 C CNN
+F 2 "" H 12250 4450 50  0000 C CNN
+F 3 "" H 12250 4450 50  0000 C CNN
+	1    12250 4450
+	0    -1   -1   0
+$EndComp
 $EndSCHEMATC

Commit message: added space savings of BoSL PCB
Parts:
- Y1: footprint Crystal:Crystal_HC49-4H_Vertical -> Crystal:Crystal_SMD_5032-2Pin_5.0x3.2mm
Changed lines of the file:
@@
 F 0 "Y1" H 4550 4450 50  0000 C CNN
 F 1 "8 MHz" H 4550 4150 50  0000 C CNN
-F 2 "Crystal:Crystal_HC49-4H_Vertical" H 4550 4300 50  0001 C CNN
+F 2 "Crystal:Crystal_SMD_5032-2Pin_5.0x3.2mm" H 4550 4300 50  0001 C CNN
 F 3 "" H 4550 4300 50  0000 C CNN
 	1    4550 4300

Commit message: updated bosl with small screw terminals
Parts:
- removed P1: CONN_01X16, Connector_PinHeader_2.54mm:PinHeader_1x16_P2.54mm_Vertical, symbol SIM7000-rescue:CONN_01X16-SIM7000-rescue
- removed P6: CONN_01X09, Connector_PinHeader_2.54mm:PinHeader_1x09_P2.54mm_Vertical, symbol SIM7000-rescue:CONN_01X09-SIM7000-rescue
- removed P9: CONN_01X12, Connector_PinHeader_2.54mm:PinHeader_1x12_P2.54mm_Vertical, symbol SIM7000-rescue:CONN_01X12-SIM7000-rescue
- added AT3: AT-GNSS, Connector_Coaxial:U.FL_Molex_MCRF_73412-0110_Vertical, symbol SIM7000-rescue:AT-ant
- added J10: Conn_01x08, symbol Connector_Generic:Conn_01x08
- added J8: Conn_01x05, Connector_PinHeader_2.54mm:PinHeader_1x05_P2.54mm_Vertical, symbol Connector_Generic:Conn_01x05
- added J9: Conn_01x06, Connector_PinHeader_2.54mm:PinHeader_1x06_P2.54mm_Vertical, symbol Connector_Generic:Conn_01x06
- J1: footprint TerminalBlock_Phoenix:TerminalBlock_Phoenix_MKDS-1,5-6_1x06_P5.00mm_Horizontal -> TerminalBlock_Phoenix:TerminalBlock_Phoenix_PT-1,5-6-3.5-H_1x06_P3.50mm_Horizontal
- J2, J5: footprint TerminalBlock_Phoenix:TerminalBlock_Phoenix_MKDS-1,5-4_1x04_P5.00mm_Horizontal -> TerminalBlock_Phoenix:TerminalBlock_Phoenix_PT-1,5-4-3.5-H_1x04_P3.50mm_Horizontal
- J3: footprint TerminalBlock_Phoenix:TerminalBlock_Phoenix_MKDS-1,5-2_1x02_P5.00mm_Horizontal -> TerminalBlock_Phoenix:TerminalBlock_Phoenix_PT-1,5-2-3.5-H_1x02_P3.50mm_Horizontal
- J4: footprint TerminalBlock_Phoenix:TerminalBlock_Phoenix_MKDS-1,5-8_1x08_P5.00mm_Horizontal -> TerminalBlock_Phoenix:TerminalBlock_Phoenix_PT-1,5-8-3.5-H_1x08_P3.50mm_Horizontal
Connections:
- net A0: now also J9.6 (Pin_6)
- net A1: now also J9.5 (Pin_5)
- net A2: now also J9.4 (Pin_4)
- net A3: now also J9.3 (Pin_3)
- net AREF: now also J8.5 (Pin_5)
- net D2: now also J10.1 (Pin_1)
- net D3: now also J10.2 (Pin_2)
- net D6: now also J10.3 (Pin_3)
- net D7: now also J10.4 (Pin_4)
- net GND: now also J5.1, AT3.2, J8.1 (Pin_1), J8.3 (Pin_3); no longer J5.4
- net SCL: now also J9.1 (Pin_1)
- net SDA: now also J9.2 (Pin_2)
- net SD_CS: now also J10.5 (Pin_5)
- net SD_MISO: now also J10.7 (Pin_7)
- net SD_MOSI: now also J10.6 (Pin_6)
- net SD_SCLK: now also J10.8 (Pin_8)
- net VPP: now also J5.2, J8.2 (Pin_2); no longer J5.1
- net V_3.3: now also J5.4, J8.4 (Pin_4); no longer J5.2
- net at AT1.1, IC2.60 (RF_ANT): now also AT3.1
Other:
- note added: "TODO:\nextra mixroaxial antenna\npressure sensor on back\nscrew terminals small"

Commit message: finished bosl rev0.4
Other:
- note removed: "TODO:\nextra mixroaxial antenna\npressure sensor on back\nscrew terminals small"
Changed lines of the file:
@@
 	0    -1   -1   0
 $EndComp
-Text Notes 5650 6950 0    60   ~ 0
-TODO:\nextra mixroaxial antenna\npressure sensor on back\nscrew terminals small
 $Comp
 L SIM7000-rescue:AT-ant AT3
