File: EDA/EDA/BoSL.kicad_pcb (KiCad board)
At the start: 2 copper layers, 79 x 69.8 mm, 67 parts, among them CON1 Micro_SD_Card, CON2 BARREL_JACK, IC2 SIM7000, J1 Screw_Terminal_1x06, J10 Conn_01x08, J2 Screw_Terminal_1x04, J3 Screw_Terminal_1x02, J4 Screw_Terminal_1x08, J5 Screw_Terminal_1x04, J6 RJ45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

Commit message: added max voltage text to bosl board on input
Parts:
- moved G1 4.30 mm to (144.9, 99.2)
Other:
- board text added: "4.5V MAX"
- board text added: "Rev: 0.4.2 Monash BoSL Board"
- board text removed: "Rev: 0.4.1 Monash BoSL Board"
Changed lines of the file:
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@@
   (general
     (thickness 1.6)
-    (drawings 88)
+    (drawings 89)
     (tracks 1027)
     (zones 0)
@@
   (title_block
     (title "Monash BoSL Board")
-    (date 2020-06-15)
-    (rev 0.4.1)
+    (date 2020-11-27)
+    (rev 0.4.2)
   )
   (layers
@@
   )
   (setup
-    (last_trace_width 0.4)
+    (last_trace_width 0.25)
     (user_trace_width 0.4)
     (user_trace_width 0.6)
@@
       (drillshape 0)
       (scaleselection 1)
-      (outputdirectory "../Manufacturing/Gerber/"))
+      (outputdirectory "Production/"))
   )
   (net 0 "")
@@
   )
   (module SIMFootprints:BoSL_Graphic (layer B.Cu)
-    (at 140.6 99.2 270)
+    (at 144.9 99.2 270)
     (fp_text reference G1 (at 0 0 90) (layer B.SilkS) hide
       (effects (font (size 1.524 1.524) (thickness 0.3)) (justify mirror))
@@
       (net 5 "Net-(C4-Pad2)"))
   )
+  (gr_text "4.5V MAX" (at 134.9 89.4 90) (layer B.SilkS)
+    (effects (font (size 1 1) (thickness 0.15)) (justify mirror))
+  )
   (gr_text RX (at 160.4 100) (layer B.SilkS)
     (effects (font (size 1 1) (thickness 0.15)) (justify mirror))
@@
     (effects (font (size 1 1) (thickness 0.15)) (justify mirror))
   )
-  (gr_text "USB PWR" (at 150.8 100) (layer B.SilkS)
+  (gr_text "USB\nPWR" (at 153.2 101.1) (layer B.SilkS)
     (effects (font (size 1 1) (thickness 0.15)) (justify mirror))
   )
@@
   (gr_line (start 192.5 130.7) (end 192.5 130.8) (layer Edge.Cuts) (width 0.15))
   (gr_line (start 192.5 129.5) (end 192.5 130.7) (layer Edge.Cuts) (width 0.15))
-  (gr_text "Rev: 0.4.1\nMonash BoSL Board" (at 187.95 64.2 90) (layer B.SilkS)
+  (gr_text "Rev: 0.4.2\nMonash BoSL Board" (at 187.95 64.2 90) (layer B.SilkS)
     (effects (font (size 2 2) (thickness 0.45)) (justify left mirror))
   )
