File: EDA/EDA/BoSL.sch (KiCad schematic (older format))
At the start: 67 parts, among them CON1 Micro_SD_Card, CON2 BARREL_JACK, IC2 SIM7000, J1 Screw_Terminal_1x06, J10 Conn_01x08, J2 Screw_Terminal_1x04, J3 Screw_Terminal_1x02, J4 Screw_Terminal_1x08, J5 Screw_Terminal_1x04, J6 RJ45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

Commit message: added snazy schematic
Parts:
- removed P2, P3, P4: CONN_01X04, Connector_PinHeader_2.54mm:PinHeader_1x04_P2.54mm_Vertical, symbol SIM7000-rescue:CONN_01X04-SIM7000-rescue
- added P2, P3: I2C, Connector_PinHeader_2.54mm:PinHeader_1x04_P2.54mm_Vertical, symbol Connector_Generic:Conn_01x04
- added P4: Serial, Connector_PinHeader_2.54mm:PinHeader_1x04_P2.54mm_Vertical, symbol Connector_Generic:Conn_01x04
- J1: value Screw_Terminal_1x06 -> Analogue
- J10: value Conn_01x08 -> Digital
- J2: value Screw_Terminal_1x04 -> I2C
- J3: value Screw_Terminal_1x02 -> Serial
- J4: value Screw_Terminal_1x08 -> Digital
- J5: value Screw_Terminal_1x04 -> Power
- J8: value Conn_01x05 -> Power
- J9: value Conn_01x06 -> Analogue
- TP4: value TestPoint -> USB_VBUS
- TP5: value TestPoint -> DM
- TP6: value TestPoint -> DP
- TP7: value TestPoint -> GND
- U6: value ATmega328P-AU -> ATmega328P
Connections:
- net GND: now also P2.3 (Pin_3), P3.3 (Pin_3), P4.4 (Pin_4)
- net SCL: now also P2.1 (Pin_1), P3.1 (Pin_1)
- net SDA: now also P2.2 (Pin_2), P3.2 (Pin_2)
- net TLL_RST: now also P4.3 (Pin_3)
- net TLL_RX: now also P4.2 (Pin_2)
- net TLL_TX: now also P4.1 (Pin_1)
- net V_3.3: now also P2.4 (Pin_4), P3.4 (Pin_4)
- net at C3.2, U6.8 (XTAL2/PB7): now also Y1.2; no longer Y1.1
- net at C2.2, U6.7 (XTAL1/PB6): now also Y1.1; no longer Y1.2
- net DM: no longer names the net of IC2.28 (USB_DM), TP5.1
- net DP: no longer names the net of IC2.27 (USB_DP), TP6.1
- net USB_VBUS: no longer names the net of IC2.24 (USB_VBUS), TP4.1
- no-connect marks 38 -> 43
Other:
- note added: "MCU ATmega328P"
- note added: "MCU Reset"
- moved on the sheet: BT1, C11, C12, C2, C3, C4, C5, C6, C7, C8, C9, D4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
